Commit message: add wheels

File: src/my_robot/urdf/my_robot.xacro (robot description, xacro)
@@ -6,4 +6,22 @@
     <parent link="robot_footprint"/>
     <child link="chassis" />
+  </joint>
+  <!-- left wheel -->
+  <joint type="continuous" name="left_wheel_hinge">
+    <origin xyz="0 0.15 0" rpy="0 0 0"/>
+    <child link="left_wheel"/>
+    <parent link="chassis"/>
+    <axis xyz="0 1 0" rpy="0 0 0"/>
+    <limit effort="10000" velocity="1000"/>
+    <dynamics damping="1.0" friction="1.0"/>
+  </joint>
+  <!-- right wheel -->
+  <joint type="continuous" name="right_wheel_hinge">
+    <origin xyz="0 -0.15 0" rpy="0 0 0"/>
+    <child link="right_wheel"/>
+    <parent link="chassis"/>
+    <axis xyz="0 1 0" rpy="0 0 0"/>
+    <limit effort="10000" velocity="1000"/>
+    <dynamics damping="1.0" friction="1.0"/>
   </joint>
   <link name='chassis'>
@@ -55,3 +73,51 @@
     </visual>
   </link>
+  <!-- left wheel -->
+  <link name='left_wheel'>
+  <inertial>
+    <mass value="5.0"/>
+    <origin xyz="0.0 0 0" rpy=" 0 0 0"/>
+    <inertia
+        ixx="0.1" ixy="0" ixz="0"
+        iyy="0.1" iyz="0"
+        izz="0.1"
+    />
+    </inertial>
+    <collision name='collision'>
+      <origin xyz="0 0 0" rpy=" 0 1.5707 1.5707"/>
+      <geometry>
+        <cylinder radius="0.1" length="0.05"/>
+      </geometry>
+    </collision>
+    <visual name='wheel_visual'>
+      <origin xyz="0 0 0" rpy=" 0 1.5707 1.5707"/>
+      <geometry>
+        <cylinder radius="0.1" length="0.05"/>
+      </geometry>
+    </visual>
+  </link>
+  <!-- rigth wheel -->
+  <link name='right_wheel'>
+  <inertial>
+    <mass value="5.0"/>
+    <origin xyz="0.0 0 0" rpy=" 0 0 0"/>
+    <inertia
+        ixx="0.1" ixy="0" ixz="0"
+        iyy="0.1" iyz="0"
+        izz="0.1"
+    />
+    </inertial>
+    <collision name='collision'>
+      <origin xyz="0 0 0" rpy=" 0 1.5707 1.5707"/>
+      <geometry>
+        <cylinder radius="0.1" length="0.05"/>
+      </geometry>
+    </collision>
+    <visual name='wheel_visual'>
+      <origin xyz="0 0 0" rpy=" 0 1.5707 1.5707"/>
+      <geometry>
+        <cylinder radius="0.1" length="0.05"/>
+      </geometry>
+    </visual>
+  </link>
 </robot>

Commit message: add lydar

File: src/my_robot/urdf/my_robot.xacro (robot description, xacro)
@@ -7,5 +7,5 @@
     <child link="chassis" />
   </joint>
-  <!-- left wheel -->
+  <!-- joint left wheel -->
   <joint type="continuous" name="left_wheel_hinge">
     <origin xyz="0 0.15 0" rpy="0 0 0"/>
@@ -16,5 +16,5 @@
     <dynamics damping="1.0" friction="1.0"/>
   </joint>
-  <!-- right wheel -->
+  <!-- joint right wheel -->
   <joint type="continuous" name="right_wheel_hinge">
     <origin xyz="0 -0.15 0" rpy="0 0 0"/>
@@ -24,4 +24,18 @@
     <limit effort="10000" velocity="1000"/>
     <dynamics damping="1.0" friction="1.0"/>
+  </joint>
+  <!-- joint camera -->
+  <joint type="fixed" name="camera_joint">
+    <origin xyz="0.2 0 0" rpy="0 0 0"/>
+    <child link="camera"/>
+    <parent link="chassis"/>
+    <axis xyz="0 1 0" rpy="0 0 0"/>
+  </joint>
+  <!-- joint hokuyo -->
+  <joint type="fixed" name="hokuyo_joint">
+    <origin xyz="0.15 0 0.1" rpy="0 0 0"/>
+    <child link="hokuyo"/>
+    <parent link="chassis"/>
+    <axis xyz="0 1 0" rpy="0 0 0"/>
   </joint>
   <link name='chassis'>
@@ -84,5 +98,5 @@
     />
     </inertial>
-    <collision name='collision'>
+    <collision name='left_wheel_collision'>
       <origin xyz="0 0 0" rpy=" 0 1.5707 1.5707"/>
       <geometry>
@@ -99,14 +113,14 @@
   <!-- rigth wheel -->
   <link name='right_wheel'>
-  <inertial>
-    <mass value="5.0"/>
-    <origin xyz="0.0 0 0" rpy=" 0 0 0"/>
-    <inertia
-        ixx="0.1" ixy="0" ixz="0"
-        iyy="0.1" iyz="0"
-        izz="0.1"
-    />
-    </inertial>
-    <collision name='collision'>
+    <inertial>
+      <mass value="5.0"/>
+      <origin xyz="0.0 0 0" rpy=" 0 0 0"/>
+      <inertia
+          ixx="0.1" ixy="0" ixz="0"
+          iyy="0.1" iyz="0"
+          izz="0.1"
+      />
+      </inertial>
+    <collision name='right_wheel_collision'>
       <origin xyz="0 0 0" rpy=" 0 1.5707 1.5707"/>
       <geometry>
@@ -121,3 +135,48 @@
     </visual>
   </link>
+  <!-- camera -->
+  <link name="camera">
+    <inertia>
+      <mass value="0.1"/>
+      <origin xyz="0.05 0.05 0.05" rpy="0 0 0"/>
+      <inertia
+          ixx="1e-6" ixy="0" ixz="0"
+          iyy="1e-6" iyz="0"
+          izz="1e-6"
+      />
+    </inertia>
+    <collision name='camera_collision'>
+      <origin xyz="0 0 0" rpy="0 0 0"/>
+      <geometry>
+        <box size="0.05 0.05 0.05"/>
+      </geometry>
+    </collision>
+    <visual name='camera_visual'>
+      <origin xyz="0 0 0" rpy="0 0 0"/>
+      <geometry>
+        <box size="0.05 0.05 0.05"/>
+      </geometry>
+    </visual>
+  </link>
+  <link name="hokuyo">
+    <inertia>
+      <mass value="1e-5"/>
+      <origin xyz="0 0 0" rpy="0 0 0"/>
+      <inertia
+          ixx="1e-6" ixy="0" ixz="0"
+          iyy="1e-6" iyz="0"
+          izz="1e-6"
+      />
+    </inertia>
+    <collision name='hokuyo_collision'>
+      <origin xyz="0 0 0" rpy="0 0 0"/>
+      <geometry>
+        <box size="0.1 0.1 0.1"/>
+      </geometry>
+    </collision>
+    <visual name='hokuyo_visual'>
+      <origin xyz="0 0 0" rpy="0 0 0"/>
+      <geometry filename = "package://my_robot/meshes/hokuyo.dae"/>
+     </visual>
+  </link>
 </robot>

Commit message: lidar meshes not working

File: src/my_robot/urdf/my_robot.xacro (robot description, xacro)
@@ -177,5 +177,5 @@
     <visual name='hokuyo_visual'>
       <origin xyz="0 0 0" rpy="0 0 0"/>
-      <geometry filename = "package://my_robot/meshes/hokuyo.dae"/>
+      <geometry filename='package://my_robot/meshes/hokuyo.dae'/>
      </visual>
   </link>

Commit message: mesh working

File: src/my_robot/urdf/my_robot.xacro (robot description, xacro)
@@ -6,36 +6,4 @@
     <parent link="robot_footprint"/>
     <child link="chassis" />
-  </joint>
-  <!-- joint left wheel -->
-  <joint type="continuous" name="left_wheel_hinge">
-    <origin xyz="0 0.15 0" rpy="0 0 0"/>
-    <child link="left_wheel"/>
-    <parent link="chassis"/>
-    <axis xyz="0 1 0" rpy="0 0 0"/>
-    <limit effort="10000" velocity="1000"/>
-    <dynamics damping="1.0" friction="1.0"/>
-  </joint>
-  <!-- joint right wheel -->
-  <joint type="continuous" name="right_wheel_hinge">
-    <origin xyz="0 -0.15 0" rpy="0 0 0"/>
-    <child link="right_wheel"/>
-    <parent link="chassis"/>
-    <axis xyz="0 1 0" rpy="0 0 0"/>
-    <limit effort="10000" velocity="1000"/>
-    <dynamics damping="1.0" friction="1.0"/>
-  </joint>
-  <!-- joint camera -->
-  <joint type="fixed" name="camera_joint">
-    <origin xyz="0.2 0 0" rpy="0 0 0"/>
-    <child link="camera"/>
-    <parent link="chassis"/>
-    <axis xyz="0 1 0" rpy="0 0 0"/>
-  </joint>
-  <!-- joint hokuyo -->
-  <joint type="fixed" name="hokuyo_joint">
-    <origin xyz="0.15 0 0.1" rpy="0 0 0"/>
-    <child link="hokuyo"/>
-    <parent link="chassis"/>
-    <axis xyz="0 1 0" rpy="0 0 0"/>
   </joint>
   <link name='chassis'>
@@ -111,4 +79,13 @@
     </visual>
   </link>
+  <!-- joint left wheel -->
+  <joint type="continuous" name="left_wheel_hinge">
+    <origin xyz="0 0.15 0" rpy="0 0 0"/>
+    <child link="left_wheel"/>
+    <parent link="chassis"/>
+    <axis xyz="0 1 0" rpy="0 0 0"/>
+    <limit effort="10000" velocity="1000"/>
+    <dynamics damping="1.0" friction="1.0"/>
+  </joint>
   <!-- rigth wheel -->
   <link name='right_wheel'>
@@ -135,4 +112,13 @@
     </visual>
   </link>
+  <!-- joint right wheel -->
+  <joint type="continuous" name="right_wheel_hinge">
+    <origin xyz="0 -0.15 0" rpy="0 0 0"/>
+    <child link="right_wheel"/>
+    <parent link="chassis"/>
+    <axis xyz="0 1 0" rpy="0 0 0"/>
+    <limit effort="10000" velocity="1000"/>
+    <dynamics damping="1.0" friction="1.0"/>
+  </joint>
   <!-- camera -->
   <link name="camera">
@@ -159,4 +145,12 @@
     </visual>
   </link>
+  <!-- joint camera -->
+  <joint type="fixed" name="camera_joint">
+    <origin xyz="0.2 0 0" rpy="0 0 0"/>
+    <child link="camera"/>
+    <parent link="chassis"/>
+    <axis xyz="0 1 0" rpy="0 0 0"/>
+  </joint>
+  <!-- hoyuko -->
   <link name="hokuyo">
     <inertia>
@@ -172,11 +166,20 @@
       <origin xyz="0 0 0" rpy="0 0 0"/>
       <geometry>
-        <box size="0.1 0.1 0.1"/>
+      <mesh filename='package://my_robot/meshes/hokuyo.dae'/>
       </geometry>
     </collision>
     <visual name='hokuyo_visual'>
       <origin xyz="0 0 0" rpy="0 0 0"/>
-      <geometry filename='package://my_robot/meshes/hokuyo.dae'/>
+      <geometry>
+        <mesh filename='package://my_robot/meshes/hokuyo.dae'/>
+      </geometry>
      </visual>
   </link>
+  <!-- joint hokuyo -->
+  <joint type="fixed" name="hokuyo_joint">
+    <origin xyz="0.15 0 0.1" rpy="0 0 0"/>
+    <child link="hokuyo"/>
+    <parent link="chassis"/>
+    <axis xyz="0 1 0" rpy="0 0 0"/>
+  </joint>
 </robot>

Commit message: colors not working

File: src/my_robot/urdf/my_robot.xacro (robot description, xacro)
@@ -29,4 +29,7 @@
         <box size=".4 .2 .1"/>
       </geometry>
+      <material name="blue">
+        <color rgba="0 0 0.8 1"/>
+      </material>
     </visual>
     <collision name='back_caster_collision'>
@@ -77,4 +80,7 @@
         <cylinder radius="0.1" length="0.05"/>
       </geometry>
+      <material name="blue">
+        <color rgba="0 0 0.8 1"/>
+     </material>
     </visual>
   </link>
@@ -110,4 +116,7 @@
         <cylinder radius="0.1" length="0.05"/>
       </geometry>
+      <material name="blue">
+        <color rgba="0 0 0.8 1"/>
+      </material>
     </visual>
   </link>

Commit message: fix number parsing

File: src/my_robot/urdf/my_robot.xacro (robot description, xacro)
@@ -22,5 +22,5 @@
       <origin xyz="0 0 0" rpy=" 0 0 0"/>
       <geometry>
-        <box size=".4 .2 .1"/>
+        <box size="0.4 0.2 0.1"/>
       </geometry>
     </collision>
@@ -28,5 +28,5 @@
       <origin xyz="0 0 0" rpy=" 0 0 0"/>
       <geometry>
-        <box size=".4 .2 .1"/>
+        <box size="0.4 0.2 0.1"/>
       </geometry>
       <material name="blue">

Commit message: add joint

File: src/my_robot/urdf/my_robot.xacro (robot description, xacro)
@@ -162,4 +162,11 @@
     <axis xyz="0 1 0" rpy="0 0 0"/>
   </joint>
+ <joint name="camera_optical_joint" type="fixed">
+    <origin xyz="0 0 0" rpy="-1.5707 0 -1.5707"/>
+    <parent link="camera_link"/>
+    <child link="camera_link_optical"/>
+  </joint>
+  <link name="camera_link_optical">
+  </link>
   <!-- hoyuko -->
   <link name="hokuyo">

Commit message: fix link v2

File: src/my_robot/urdf/my_robot.xacro (robot description, xacro)
@@ -162,11 +162,10 @@
     <axis xyz="0 1 0" rpy="0 0 0"/>
   </joint>
- <joint name="camera_optical_joint" type="fixed">
+  <link name="camera_link_optical"></link>
+  <joint name="camera_optical_joint" type="fixed">
     <origin xyz="0 0 0" rpy="-1.5707 0 -1.5707"/>
     <parent link="camera_link"/>
     <child link="camera_link_optical"/>
   </joint>
-  <link name="camera_link_optical">
-  </link>
   <!-- hoyuko -->
   <link name="hokuyo">

Commit message: change camera link 4

File: src/my_robot/urdf/my_robot.xacro (robot description, xacro)
@@ -165,5 +165,5 @@
   <joint name="camera_optical_joint" type="fixed">
     <origin xyz="0 0 0" rpy="-1.5707 0 -1.5707"/>
-    <parent link="camera_link"/>
+    <parent link="camera"/>
     <child link="camera_link_optical"/>
   </joint>

Commit message: fixes

File: src/my_robot/urdf/my_robot.xacro (robot description, xacro)
@@ -132,8 +132,8 @@
   </joint>
   <!-- camera -->
-  <link name="camera">
-    <inertia>
+    <link name="camera">
+    <inertial>
       <mass value="0.1"/>
-      <origin xyz="0.05 0.05 0.05" rpy="0 0 0"/>
+      <origin xyz="0.0 0 0" rpy=" 0 0 0"/>
       <inertia
           ixx="1e-6" ixy="0" ixz="0"
@@ -141,7 +141,7 @@
           izz="1e-6"
       />
-    </inertia>
-    <collision name='camera_collision'>
-      <origin xyz="0 0 0" rpy="0 0 0"/>
+    </inertial>
+    <collision name='collision'>
+      <origin xyz="0.0 0 0" rpy=" 0 0 0"/>
       <geometry>
         <box size="0.05 0.05 0.05"/>
@@ -149,5 +149,5 @@
     </collision>
     <visual name='camera_visual'>
-      <origin xyz="0 0 0" rpy="0 0 0"/>
+      <origin xyz="0.0 0 0" rpy=" 0 0 0"/>
       <geometry>
         <box size="0.05 0.05 0.05"/>
@@ -155,16 +155,17 @@
     </visual>
   </link>
-  <!-- joint camera -->
   <joint type="fixed" name="camera_joint">
-    <origin xyz="0.2 0 0" rpy="0 0 0"/>
+    <origin xyz="0.35 0 0" rpy="0 0 0"/>
     <child link="camera"/>
     <parent link="chassis"/>
     <axis xyz="0 1 0" rpy="0 0 0"/>
-  </joint>
-  <link name="camera_link_optical"></link>
-  <joint name="camera_optical_joint" type="fixed">
-    <origin xyz="0 0 0" rpy="-1.5707 0 -1.5707"/>
+    <limit effort="10000" velocity="1000"/>
+    <dynamics damping="1.0" friction="1.0"/>
+  </joint>
+  <link name="camera_rgbd_frame"></link>
+  <joint name="camera_rgbd_joint" type="fixed">
+    <origin xyz="0 0 0" rpy="-${pi/2} 0 -${pi/2}"/>
     <parent link="camera"/>
-    <child link="camera_link_optical"/>
+    <child link="camera_rgbd_frame"/>
   </joint>
   <!-- hoyuko -->

Commit message: make ready for submission

File: src/my_robot/urdf/my_robot.xacro (robot description, xacro)
@@ -163,5 +163,4 @@
     <dynamics damping="1.0" friction="1.0"/>
   </joint>
-  <link name="camera_rgbd_frame"></link>
   <joint name="camera_rgbd_joint" type="fixed">
     <origin xyz="0 0 0" rpy="-${pi/2} 0 -${pi/2}"/>
@@ -169,4 +168,5 @@
     <child link="camera_rgbd_frame"/>
   </joint>
+  <link name="camera_rgbd_frame"></link>
   <!-- hoyuko -->
   <link name="hokuyo">

Commit message: add model an move camera

File: src/my_robot/urdf/my_robot.xacro (robot description, xacro)
@@ -156,5 +156,5 @@
   </link>
   <joint type="fixed" name="camera_joint">
-    <origin xyz="0.35 0 0" rpy="0 0 0"/>
+    <origin xyz="0 0 0" rpy="0 0 0"/>
     <child link="camera"/>
     <parent link="chassis"/>
@@ -164,5 +164,5 @@
   </joint>
   <joint name="camera_rgbd_joint" type="fixed">
-    <origin xyz="0 0 0" rpy="-${pi/2} 0 -${pi/2}"/>
+    <origin xyz="0 0 0" rpy="0 0 0"/>
     <parent link="camera"/>
     <child link="camera_rgbd_frame"/>
